File: PLC Sanit industries/PLC Sanit industries.kicad_pcb (KiCad board)
At the start: 2 copper layers, 215 x 111.3 mm, 0 parts

Commit message: rfghjkl
Parts:
- added R40: 4.7k, Resistor_SMD:R_0805_2012Metric_Pad1.20x1.40mm_HandSolder, F.Cu at (108.5, 48.0)
Routing:
- net gnd: track 0.00 -> 262.6 mm, vias 0 -> 104
- net (no net): track 6501.8 -> 6250.2 mm, vias 317 -> 215

Commit message: sdffghjhkl
Parts:
- added REF**: RJ14_Connfly_DS1133-S4_Horizontal, Connector_RJ:RJ14_Connfly_DS1133-S4_Horizontal, F.Cu at (75.5, 50.3)
- added REF**: RJ14_Connfly_DS1133-S4_Horizontal, Connector_RJ:RJ14_Connfly_DS1133-S4_Horizontal, F.Cu at (91.0, 50.3)
Routing:
- net (no net): track 6250.2 -> 5374.8 mm, vias 215 -> 184
- net vcc: track 0.00 -> 692.7 mm, vias 0 -> 20
- net rx: track 0.00 -> 183.7 mm, vias 0 -> 6
- net tx: track 0.00 -> 98.5 mm, vias 0 -> 6
- net gnd: track 262.6 -> 268.1 mm

Commit message: sdffghjhkl
Parts:
- added REF**: FanPinHeader_1x04_P2.54mm_Vertical, Connector:FanPinHeader_1x04_P2.54mm_Vertical, F.Cu at (138.0, 75.6)
Routing:
- net (no net): track 5374.8 -> 5159.3 mm, vias 184 -> 172
- net scl: track 0.00 -> 117.1 mm, vias 0 -> 5
- net sda: track 0.00 -> 98.4 mm, vias 0 -> 5
- net gnd: track 268.1 -> 273.0 mm, vias 104 -> 103
- net vcc: vias 20 -> 19
Other:
- board text added: "Q2"
