File: RejsaCAN board/RejsaCAN board/RejsaCAN board.kicad_pcb (KiCad board)
At the start: 2 copper layers, 1 part

Commit message: dtfgkhfdftfvuyfu
Parts:
- removed REF**: JST_B8B-XH-A, JST XH:CONN 8 JST_B8B-XH-A
- added C1: 100uF, SD-CARD-MEM2075-00-140-01-A:SD-CARD-MEM2075-00-140-01-A, F.Cu at (8.43, 12.7)
- added C10: 22uF, Capacitor_SMD:C_0201_0603Metric, F.Cu at (102.6, 134.6)
- added C11: 22uF, Capacitor_SMD:C_0201_0603Metric, F.Cu at (162.2, 102.6)
- added C12: 100nF, Capacitor_SMD:C_0201_0603Metric, F.Cu at (115.1, 132.4)
- added C13: 100nF, Capacitor_SMD:C_0201_0603Metric, F.Cu at (102.4, 118.8)
- added C14: 10uF, Capacitor_SMD:C_0201_0603Metric, F.Cu at (102.4, 120.8)
- added C15: 1uF, Capacitor_SMD:C_0201_0603Metric, F.Cu at (102.4, 114.5)
- added C16: 12uF, Capacitor_SMD:C_0201_0603Metric, F.Cu at (143.5, 127.3)
- added C17: 12uF, Capacitor_SMD:C_0201_0603Metric, F.Cu at (115.1, 130.0)
- added C2: 100uF, Capacitor_SMD:C_0201_0603Metric, F.Cu at (162.2, 103.6)
- added C3: 1uF, Capacitor_SMD:C_0201_0603Metric, F.Cu at (163.8, 102.3)
- added C4: 100nF, Capacitor_SMD:C_0201_0603Metric, F.Cu at (102.6, 130.5)
- added C5: 1uF, Capacitor_SMD:C_0201_0603Metric, F.Cu at (109.6, 109.1)
- added C6: 1uF, Capacitor_SMD:C_0201_0603Metric, F.Cu at (102.4, 116.8)
- added C7: 100nF, Capacitor_SMD:C_0201_0603Metric, F.Cu at (112.4, 106.8)
- added C8: 22uF, Capacitor_SMD:C_0201_0603Metric, F.Cu at (102.6, 132.5)
- added C9: 22uF, Capacitor_SMD:C_0201_0603Metric, F.Cu at (102.6, 128.3)
- added D1: GREEN, LED_SMD:LED_0201_0603Metric, F.Cu at (143.6, 117.0)
- added D10: 1N4148W, Diode_SMD:D_SOD-123, F.Cu at (153.0, 100.2)
- added D11: SS34, Diode_SMD:D_SMA, F.Cu at (120.0, 131.0)
- added D12: LED, LED_SMD:LED_0201_0603Metric, F.Cu at (124.7, 123.9)
- added D13: SS14, Diode_SMD:D_SMA, F.Cu at (139.6, 110.3)
- added D14: 1N4148W, Diode_SMD:D_SOD-123, F.Cu at (153.1, 103.2)
- added D15: 1N4148W, Diode_SMD:D_SOD-123, F.Cu at (149.8, 107.2)
- added D17: SMF30A, Diode_SMD:D_SMF, F.Cu at (106.2, 107.9)
- added D2: BLUE, LED_SMD:LED_0201_0603Metric, F.Cu at (143.6, 119.0)
- added D3: YELLOW, LED_SMD:LED_0201_0603Metric, F.Cu at (143.6, 118.0)
- added D4: SS34, Diode_SMD:D_SMA, F.Cu at (141.7, 142.4)
- added D5: SS34, Diode_SMD:D_SMA, F.Cu at (133.6, 142.3)
- added D6: ESD9B5.0ST5G, Diode_SMD:D_SOD-923, F.Cu at (164.8, 131.3)
- added D7: ESD9B5.0ST5G, Diode_SMD:D_SOD-923, F.Cu at (164.8, 132.8)
- added D8: ESD9B5.0ST5G, Diode_SMD:D_SOD-923, F.Cu at (164.8, 134.3)
- added D9: 1N4148W, Diode_SMD:D_SOD-123, F.Cu at (153.0, 97.5)
- added F1: Fuse_Small, Fuse:Fuse_0402_1005Metric, F.Cu at (129.0, 123.9)
- added J1: B8B-XH-A, JST XH:CONN 8 JST_B8B-XH-A, F.Cu at (149.6, 136.8)
- added J10: B8B-XH-A, JST XH:CONN 8 JST_B8B-XH-A, F.Cu at (125.5, 136.8)
- added J8: Connector, USB-TYPE-C-16P, PCM_JLCPCB:TYPE-C-SMD_HX-TYPE-C-16PIN, F.Cu at (143.4, 101.1)
- added J9: B8B-XH-A, JST XH:CONN 8 JST_B8B-XH-A, F.Cu at (109.5, 124.5)
- added L1: 10uH, Inductor_SMD:L_Neosid_SM-PIC0512H, F.Cu at (128.4, 128.2)
- added L2: 22uH, Inductor_SMD:L_Neosid_SM-PIC0512H, F.Cu at (126.4, 119.5)
- added PS1: ME2108A33P, ME2108A33P:ME2108A33P, F.Cu at (117.4, 126.1)
- added Q1: SS8050, Package_TO_SOT_SMD:SOT-23, F.Cu at (117.9, 118.4)
- added R1: 10K, Resistor_SMD:R_0201_0603Metric, F.Cu at (162.2, 101.6)
- added R10: 10K, Resistor_SMD:R_0201_0603Metric, F.Cu at (114.4, 113.8)
- added R11: 5.1K, Resistor_SMD:R_0201_0603Metric, F.Cu at (146.3, 106.5)
- added R12: 5.1K, Resistor_SMD:R_0201_0603Metric, F.Cu at (141.4, 106.1)
- added R13: 22K, Resistor_SMD:R_0201_0603Metric, F.Cu at (143.6, 116.0)
- added R14: 500, Resistor_SMD:R_0201_0603Metric, F.Cu at (143.6, 120.0)
- added R15: 1K, Resistor_SMD:R_0201_0603Metric, F.Cu at (141.7, 118.0)
- added R16: 12K, Resistor_SMD:R_0201_0603Metric, F.Cu at (146.4, 131.9)
- added R17: 10K, Resistor_SMD:R_0201_0603Metric, F.Cu at (134.9, 123.0)
- added R18: 120K, Resistor_SMD:R_0201_0603Metric, F.Cu at (142.6, 113.1)
- added R19: ADJUST, Resistor_SMD:R_0201_0603Metric, F.Cu at (108.8, 107.7)
- added R2: 22K, Resistor_SMD:R_0201_0603Metric, F.Cu at (160.5, 103.6)
- added R20: 10K, Resistor_SMD:R_0201_0603Metric, F.Cu at (142.6, 125.7)
- added R21: 10K, Resistor_SMD:R_0201_0603Metric, F.Cu at (142.6, 124.5)
- added R22: 10K, Resistor_SMD:R_0201_0603Metric, F.Cu at (136.6, 123.0)
- added R23: 10K, Resistor_SMD:R_0201_0603Metric, F.Cu at (126.9, 123.9)
- added R24: 20K, Resistor_SMD:R_0201_0603Metric, F.Cu at (127.2, 132.0)
- added R25: 20K, Resistor_SMD:R_0201_0603Metric, F.Cu at (115.1, 131.1)
- added R26: 20K, Resistor_SMD:R_0201_0603Metric, F.Cu at (142.3, 127.3)
- added R27: 10K, Resistor_SMD:R_0201_0603Metric, F.Cu at (154.4, 107.2)
- added R28: 10K, Resistor_SMD:R_0201_0603Metric, F.Cu at (153.5, 131.9)
- added R3: 120, Resistor_SMD:R_0201_0603Metric, F.Cu at (141.1, 122.8)
- added R4: 91K, Resistor_SMD:R_0201_0603Metric, F.Cu at (108.5, 106.2)
- added R5: 33K, Resistor_SMD:R_0201_0603Metric, F.Cu at (108.5, 109.1)
- added R6: 33K, Resistor_SMD:R_0201_0603Metric, F.Cu at (144.3, 113.1)
- added R7: 10K, Resistor_SMD:R_0201_0603Metric, F.Cu at (117.0, 122.1)
- added R8: ALWAYS ON JUMPER, Resistor_SMD:R_0201_0603Metric, F.Cu at (116.1, 110.4)
- added R9: 33K, Resistor_SMD:R_0201_0603Metric, F.Cu at (116.2, 114.1)
- added SD-CARD1: MEM2075-00-140-01-A, SD-CARD-MEM2075-00-140-01-A:SD-CARD-MEM2075-00-140-01-A, F.Cu at (126.5, 100.1)
- added SW1: RESET, Button_Switch_SMD:SW_Push_SPST_NO_Alps_SKRK, F.Cu at (163.8, 107.1)
- added SW2: PROG, Button_Switch_SMD:SW_Push_SPST_NO_Alps_SKRK, F.Cu at (158.1, 107.1)
- added U1: ESP32-S3-WROOM-1, RF_Module:ESP32-S3-WROOM-1, F.Cu at (159.9, 119.9)
- added U2: SN65HVD230, Package_SO:SOIC-8_3.9x4.9mm_P1.27mm, F.Cu at (136.7, 119.0)
- added U3: ~, ME2807A33M3G:ME2807A33M3G, F.Cu at (113.4, 103.5)
- added U4: LMR14206, Package_TO_SOT_SMD:SOT-23-6, F.Cu at (113.2, 109.8)
- added U5: ~, MCP9700AT-E_LT:SOT65P210X110-5N, F.Cu at (143.5, 130.9)
- added U6: MAX485E, Package_SO:SOIC-8_3.9x4.9mm_P1.27mm, F.Cu at (137.1, 127.2)
Routing:
- net GND: track 0.00 -> 323.2 mm, vias 0 -> 14
- net +3V3: track 0.00 -> 183.4 mm, vias 0 -> 11
- net MTCK: track 0.00 -> 109.8 mm, vias 0 -> 4
- net MTDI: track 0.00 -> 108.0 mm, vias 0 -> 5
- net USB5V: track 0.00 -> 86.2 mm, vias 0 -> 8
- net VCC: track 0.00 -> 81.4 mm, vias 0 -> 9
- net SDA: track 0.00 -> 77.4 mm, vias 0 -> 1
- net SCL: track 0.00 -> 76.1 mm, vias 0 -> 1
- net MTDO: track 0.00 -> 66.7 mm, vias 0 -> 2
- net 5VOLTS: track 0.00 -> 66.0 mm, vias 0 -> 7
- net Net-(D10-A): track 0.00 -> 61.5 mm
- net Net-(D10-K): track 0.00 -> 60.3 mm, vias 0 -> 2
- net USB_D-: track 0.00 -> 50.9 mm, vias 0 -> 2
- net Net-(U6-A): track 0.00 -> 48.1 mm, vias 0 -> 1
- net USB_D+: track 0.00 -> 48.0 mm, vias 0 -> 2
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Other:
- board outline added: 71.9 x 50 mm
- board text added: "+2348067136319"
- board text added: "3V3S MTCK MTDO MTDI ~B ~A GND NC"
- board text added: "48 47 16 15 12 07 06 NULL"
- board text added: "Designed by HARUNA AUWALU"
- board text added: "VCC_IN GND 3V3 SCL SDA TJ CAN_H CAN_L"
