File: ElectricSuperCar-Single-Layer LED PCB/Single-Layer LED PCB/Single-Layer LED PCB.kicad_pcb (KiCad board)
At the start: 2 copper layers, 1119.7 x 8.9 mm, 146 parts, among them J1 S3B-ZR-SM4A-TF, J2 S3B-ZR-SM4A-TF

Commit message: 6th, january. 2026
Routing:
- net VSS: track 3956.2 -> 2345.1 mm, vias 0 -> 8
- net VDD: track 1273.1 -> 1258.8 mm
Changed lines of the file:
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@@
 			(drillshape 0)
 			(scaleselection 1)
-			(outputdirectory "../../../Desktop/LED/")
+			(outputdirectory "../../../Desktop/LEDs_v3/")
 		)
 	)
@@
 	)
 	(segment
+		(start 45.6 36.4)
+		(end 43.5 36.4)
+		(width 1)
+		(layer "F.Cu")
+		(net 3)
+	)
+	(segment
 		(start 111.973501 39.400999)
 		(end 113.1745 38.2)
@@
 	)
 	(segment
+		(start 43.5 36.4)
+		(end 44.7 36.4)
+		(width 1)
+		(layer "F.Cu")
+		(net 3)
+	)
+	(segment
 		(start 863.7245 38.2)
 		(end 864.925499 39.400999)
@@
 	)
 	(segment
+		(start 1133.3 36.4)
+		(end 1134.4 36.4)
+		(width 1)
+		(layer "F.Cu")
+		(net 3)
+	)
+	(segment
 		(start 585.8745 38.2)
 		(end 587.075499 39.400999)
@@
 	)
 	(segment
+		(start 1134.4 36.4)
+		(end 1147 36.4)
+		(width 1)
+		(layer "F.Cu")
+		(net 3)
+	)
+	(segment
 		(start 922.873501 39.400999)
 		(end 924.0745 38.2)
@@
 	)
 	(segment
+		(start 39.1 36.4)
+		(end 43.5 36.4)
+		(width 1)
+		(layer "F.Cu")
+		(net 3)
+	)
+	(segment
 		(start 398.3745 38.2)
 		(end 399.575499 39.400999)
@@
 	)
 	(segment
-		(start 1127.8745 36.4)
-		(end 1147 36.4)
-		(width 1)
-		(layer "F.Cu")
-		(net 3)
-	)
-	(segment
 		(start 952.873501 39.400999)
 		(end 954.0745 38.2)
@@
 	)
 	(segment
-		(start 39.1 36.4)
-		(end 51.3745 36.4)
-		(width 1)
-		(layer "F.Cu")
-		(net 3)
-	)
-	(segment
 		(start 166.875499 39.400999)
 		(end 171.973501 39.400999)
@@
 	)
 	(segment
+		(start 1134.4 36.4)
+		(end 1134.849997 36.4)
+		(width 1)
+		(layer "F.Cu")
+		(net 3)
+	)
+	(segment
+		(start 1134.4 36.4)
+		(end 1134.099994 36.4)
+		(width 1)
+		(layer "F.Cu")
+		(net 3)
+	)
+	(segment
 		(start 69.375499 39.400999)
 		(end 74.473501 39.400999)
@@
 	)
 	(segment
+		(start 1126.1745 38.1)
+		(end 1127.8745 36.4)
+		(width 1)
+		(layer "F.Cu")
+		(net 3)
+	)
+	(segment
 		(start 449.673501 39.400999)
 		(end 450.8745 38.2)
@@
 	)
 	(segment
+		(start 44.7 36.4)
+		(end 45.3 36.4)
+		(width 0.2)
+		(layer "F.Cu")
+		(net 3)
+	)
+	(segment
 		(start 399.575499 39.400999)
 		(end 404.673501 39.400999)
@@
 	)
 	(segment
+		(start 44.7 36.4)
+		(end 45.6 36.4)
+		(width 1)
+		(layer "F.Cu")
+		(net 3)
+	)
+	(segment
 		(start 119.473501 39.400999)
 		(end 120.6745 38.2)
@@
 	)
 	(segment
+		(start 1127.8745 36.4)
+		(end 1133.3 36.4)
+		(width 1)
+		(layer "F.Cu")
+		(net 3)
+	)
+	(segment
 		(start 623.3745 38.2)
 		(end 624.575499 39.400999)
@@
 	)
 	(segment
-		(start 1126.1745 38.1)
-		(end 1127.8745 36.4)
-		(width 1)
-		(layer "F.Cu")
-		(net 3)
-	)
-	(segment
 		(start 924.0745 38.2)
 		(end 925.275499 39.400999)
@@
 	)
 	(segment
+		(start 45.6 36.4)
+		(end 51.3745 36.4)
+		(width 1)
+		(layer "F.Cu")
+		(net 3)
+	)
+	(segment
 		(start 255.7745 38.2)
 		(end 256.975499 39.400999)
@@
 		(net 3)
 	)
+	(via
+		(at 1134.099994 36.4)
+		(size 0.6)
+		(drill 0.4)
+		(layers "F.Cu" "B.Cu")
+		(net 3)
+	)
+	(via
+		(at 1134.849997 36.4)
+		(size 0.6)
+		(drill 0.4)
+		(layers "F.Cu" "B.Cu")
+		(net 3)
+	)
+	(via
+		(at 45.6 36.4)
+		(size 0.6)
+		(drill 0.4)
+		(layers "F.Cu" "B.Cu")
+		(net 3)
+	)
+	(via
+		(at 43.5 36.4)
+		(size 0.6)
+		(drill 0.4)
+		(layers "F.Cu" "B.Cu")
+		(net 3)
+	)
+	(via
+		(at 1133.3 36.4)
+		(size 0.6)
+		(drill 0.4)
+		(layers "F.Cu" "B.Cu")
+		(net 3)
+	)
+	(via
+		(at 1132.4 36.4)
+		(size 0.6)
+		(drill 0.4)
+		(layers "F.Cu" "B.Cu")
+		(net 3)
+	)
+	(via
+		(at 44.7 36.4)
+		(size 0.6)
+		(drill 0.4)
+		(layers "F.Cu" "B.Cu")
+		(net 3)
+	)
+	(via
+		(at 1135.6 36.4)
+		(size 0.6)
+		(drill 0.4)
+		(layers "F.Cu" "B.Cu")
+		(net 3)
+	)
 	(segment
-		(start 599.1 36.45)
-		(end 1140.701 36.45)
-		(width 1)
+		(start 45.65 36.45)
+		(end 45.6 36.4)
+		(width 0.2)
 		(layer "B.Cu")
 		(net 3)
@@
 	)
 	(segment
-		(start 1139.802 36.45)
-		(end 599.1 36.45)
-		(width 1)
-		(layer "B.Cu")
-		(net 3)
-	)
-	(segment
-		(start 599.1 36.45)
-		(end 1138.101 36.45)
-		(width 1)
+		(start 593.05 36.45)
+		(end 45.65 36.45)
+		(width 0.2)
 		(layer "B.Cu")
 		(net 3)
@@
 	)
 	(segment
-		(start 599.1 36.45)
-		(end 1139.8 36.45)
-		(width 1)
-		(layer "B.Cu")
-		(net 3)
-	)
-	(segment
 		(start 986.6745 34.9)
 		(end 987.8255 33.749)
@@
 	)
 	(segment
-		(start 776.0245 34.9)
-		(end 777.4755 36.351)
-		(width 1)
-		(layer "F.Cu")
-		(net 4)
-	)
-	(segment
 		(start 589.6755 33.699)
 		(end 594.7735 33.699)
@@
 	)
 	(segment
-		(start 888.9745 34.9)
-		(end 890.4255 36.351)
-		(width 1)
-		(layer "F.Cu")
-		(net 4)
-	)
-	(segment
 		(start 189.5735 33.699)
 		(end 190.7745 34.9)
@@
 	)
 	(segment
-		(start 1009.1745 34.9)
-		(end 1010.6255 36.351)
-		(width 1)
-		(layer "F.Cu")
-		(net 4)
-	)
-	(segment
 		(start 677.2735 33.699)
 		(end 678.4745 34.9)
@@
 	)
 	(segment
-		(start 258.3745 34.9)
-		(end 259.8255 36.351)
-		(width 1)
-		(layer "F.Cu")
-		(net 4)
-	)
-	(segment
 		(start 415.9745 34.9)
 		(end 417.1755 33.699)
@@
 	)
 	(segment
-		(start 363.4745 34.9)
-		(end 364.9255 36.351)
-		(width 1)
-		(layer "F.Cu")
-		(net 4)
-	)
-	(segment
 		(start 244.4755 33.699)
 		(end 249.6735 33.699)
@@
 	)
 	(segment
-		(start 994.1745 34.9)
-		(end 995.6255 36.351)
-		(width 1)
-		(layer "F.Cu")
-		(net 4)
-	)
-	(segment
 		(start 684.7735 33.699)
 		(end 679.6755 33.699)
@@
 		(width 1)
 		(layer "F.Cu")
-		(net 4)
-	)
-	(segment
-		(start 813.6745 34.9)
-		(end 815.1255 36.351)
-		(width 1)
-		(layer "F.Cu")
