File: Compact USB-C PD Sink PCB/Compact USB-C PD Sink PCB/Compact USB-C PD Sink PCB.kicad_sch (KiCad schematic)
At the start: 0 parts

Commit message: 20th, January. 2026
Parts:
- added C1, C2, C3: 10nF, PCM_JLCPCB:C_0402, symbol PCM_JLCPCB-Capacitors:0402,10nF
- added C10: 1uF, PCM_JLCPCB:C_0603, symbol PCM_JLCPCB-Capacitors:0603,1uF
- added C4, C5: 1uF, PCM_JLCPCB:C_0402, symbol PCM_JLCPCB-Capacitors:0402,1uF
- added C6, C7, C8: 10uF, PCM_JLCPCB:C_0805, symbol PCM_JLCPCB-Capacitors:0805,10uF
- added C9: 22uF, PCM_JLCPCB:C_0805, symbol PCM_JLCPCB-Capacitors:0805,22uF
- added D1, D2, D3: BAT54, PCM_JLCPCB:D_SOT-23, symbol PCM_JLCPCB-Diodes:Schottky,BAT54
- added D4, D5, D6: SMBJ5.0CA, PCM_JLCPCB:D_SMB, symbol PCM_JLCPCB-Diodes:TVS-Bi,SMBJ5.0CA
- added J1, J2, J3: Conn_01x05, Connector_Wire:SolderWire-0.1sqmm_1x05_P3.6mm_D0.4mm_OD1mm, symbol Connector_Generic:Conn_01x05
- added J5: Conn_01x06, Connector_Wire:SolderWire-0.1sqmm_1x06_P3.6mm_D0.4mm_OD1mm, symbol Connector_Generic:Conn_01x06
- added Q1, Q2, Q3: SI2301CDS-T1-GE3, PCM_JLCPCB:Q_SOT-23, symbol PCM_JLCPCB-Transistors:PMOS,SI2301CDS-T1-GE3
- added R1, R2, R3, R4, R5, R6, R7, R8, R9: 10kΩ, PCM_JLCPCB:R_0402, symbol PCM_JLCPCB-Resistors:0402,10kΩ
- added U1: STUSB4500QTR, Package_DFN_QFN:QFN-24-1EP_4x4mm_P0.5mm_EP2.7x2.7mm, symbol Interface_USB:STUSB4500QTR
- added U2, U3, U4: LM74700, Package_TO_SOT_SMD:SOT-23-6, symbol Power_Management:LM74700
- added U5: TPD2E2U06DCK, Package_TO_SOT_SMD:SOT-323_SC-70, symbol Power_Protection:TPD2E2U06DCK
Connections:
- new net: D3.1, Q3.2 (S)
- new net: R8.1, U1.20 (POWER_OK2)
- new net: R3.1, U3.3 (EN)
- new net: C4.2, U1.21 (VREG_1V2)
- new net: C5.2, U1.23 (VREG_2V7)
- new net: R4.2, U1.1 (CC1DB)
- new net: C1.1, U2.1 (VCAP)
- new net: R7.1, U1.14 (POWER_OK3)
- new net: R1.1, U2.3 (EN)
- new net: D2.1, Q2.2 (S)
- new net: D1.1, Q1.2 (S)
- new net: R2.1, U4.3 (EN)
- new net: R6.1, U1.6 (RESET)
- new net: R9.2, U1.15 (GPIO)
- new net: C2.1, U4.1 (VCAP)
- new net: C3.1, U3.1 (VCAP)
- new net: R5.2, U1.5 (CC2DB)
- new net AN/VBUS_1: C6.1, D4.1, J1.1 (Pin_1), U2.6 (ANODE)
- new net AN/VBUS_2: C7.1, D5.1, J2.1 (Pin_1), U4.6 (ANODE)
- new net AN/VBUS_3: C8.1, D6.1, J3.1 (Pin_1), U3.6 (ANODE)
- new net CATH/DRAIN_1: Q1.3 (D), U2.4 (CATHODE)
- new net CATH/DRAIN_2: Q2.3 (D), U4.4 (CATHODE)
- new net CATH/DRAIN_3: Q3.3 (D), U3.4 (CATHODE)
- new net CATH/VBUS_OR: C10.1, C9.1, D1.3, D2.3, D3.3, J5.1 (Pin_1), R6.2, U1.18 (VBUS_VS_DISCH), U1.22 (VSYS), U1.24 (VDD)
- new net GATE_1: Q1.1 (G), U2.5 (GATE)
- new net GATE_2: Q2.1 (G), U4.5 (GATE)
- new net GATE_3: Q3.1 (G), U3.5 (GATE)
- new net GND: C1.2, C10.2, C2.2, C3.2, C4.1, C5.1, C6.2, C7.2, C8.2, C9.2, D4.2, D5.2, D6.2, J1.4 (Pin_4), J1.5 (Pin_5), J2.4 (Pin_4), J2.5 (Pin_5), J3.4 (Pin_4), J3.5 (Pin_5), J5.4 (Pin_4), R1.2, R2.2, R3.2, R4.1, R5.1, R7.2, R8.2, R9.1, U1.10 (GND), U1.12 (ADDR0), U1.13 (ADDR1), U1.25 (GND), U2.2 (GND), U3.2 (GND), U4.2 (GND), U5.3
- new net I/O1/CC1: J5.5 (Pin_5), U1.2 (CC1), U5.1
- new net I/O2/CC2: J5.6 (Pin_6), U1.4 (CC2), U5.2
- no-connect marks 0 -> 15
