File: Vinicius/vinicius_device/vinicius_device.kicad_pcb (KiCad board)
At the start: 2 copper layers, 29.7 x 29.7 mm, 4 parts, among them J1 Connector, USB-TYPE-C-16P, U1 ESP32-C3, U2 CP2102-GMR, U3 VL53L0CXV0DH1

Commit message: 6th, january. 2026
Parts:
- added C1: 12pF, PCM_JLCPCB:C_0402, F.Cu at (136.8, 87.3)
- added C2: 12pF, PCM_JLCPCB:C_0402, F.Cu at (139.1, 81.4)
- added C3: 1uF, PCM_JLCPCB:C_0402, F.Cu at (148.4, 85.1)
- added C4: 1uF, PCM_JLCPCB:C_0402, F.Cu at (138.0, 91.7)
- added C5: 10uF, PCM_JLCPCB:C_0603, F.Cu at (155.0, 82.4)
- added C6: 100nF, PCM_JLCPCB:C_0402, F.Cu at (146.0, 79.9)
- added C7: 10uF, PCM_JLCPCB:C_0603, F.Cu at (152.8, 82.2)
- added D1: LTST-C191KRKT, LTST-C191KRKT:0603, F.Cu at (151.5, 86.2)
- added D2: LTST-C191KRKT, LTST-C191KRKT:0603, F.Cu at (151.5, 84.7)
- added D3: LTST-C191KRKT, LTST-C191KRKT:0603, F.Cu at (138.1, 95.2)
- added J2: U.FL, PCM_JLCPCB:IPEX-SMD_BWIPX-1-001E, F.Cu at (140.0, 89.4)
- added L1: 68nH,300mA, PCM_JLCPCB:L_0603, F.Cu at (133.3, 86.9)
- added R1: 1kΩ, PCM_JLCPCB:R_0402, F.Cu at (151.3, 81.9)
- added R10: 100kΩ, PCM_JLCPCB:R_0402, F.Cu at (148.4, 83.2)
- added R2: 1kΩ, PCM_JLCPCB:R_0402, F.Cu at (150.0, 81.9)
- added R3: 1.2kΩ, PCM_JLCPCB:R_0402, F.Cu at (154.2, 75.6)
- added R4: 100kΩ, PCM_JLCPCB:R_0402, F.Cu at (146.0, 78.8)
- added R5: 100kΩ, PCM_JLCPCB:R_0402, F.Cu at (145.4, 77.1)
- added R6: 4.7kΩ, PCM_JLCPCB:R_0402, F.Cu at (144.8, 88.0)
- added R7: 4.7kΩ, PCM_JLCPCB:R_0402, F.Cu at (143.8, 88.0)
- added R8: 330Ω, PCM_JLCPCB:R_0402, F.Cu at (151.4, 95.4)
- added REF**: SolderWire-0.1sqmm_1x02_P3.6mm_D0.4mm_OD1mm, Connector_Wire:SolderWire-0.1sqmm_1x02_P3.6mm_D0.4mm_OD1mm, F.Cu at (156.1, 77.7)
- added U4: TLV70233_SOT23-5, Package_TO_SOT_SMD:SOT-23-5, F.Cu at (155.9, 85.3)
- added U5: W25Q128, PCM_JLCPCB:SOIC-8_L5.3-W5.3-P1.27-LS8.0-BL, F.Cu at (139.7, 76.6)
- added X1: X322516MLB4SI, PCM_JLCPCB:OSC-SMD_4P-L3.2-W2.5-BL, F.Cu at (139.7, 84.0)
- U2: value CP2102-GMR -> TP4056; footprint PCM_JLCPCB:WQFN-28_L5.0-W5.0-P0.50-BL-EP3.2 -> PCM_JLCPCB:ESOP-8_L4.9-W3.9-P1.27-LS6.0-BL-EP
- moved U1 19.1 mm to (134.4, 82.5), turned to 90 degrees
- moved U2 12.5 mm to (150.6, 76.8), turned to 180 degrees
Connections:
- J1 pad A12B1: Net-(J1-GND-PadA12B1) -> BATTERY_-
- J1 pad A6: unconnected-(J1-D+-PadA6) -> USB_D+
- J1 pad A7: unconnected-(J1-D--PadA7) -> USB_D-
- J1 pad A9B4: Net-(J1-VBUS-PadA9B4) -> 5v_Input
- J1 pad B12A1: Net-(J1-GND-PadA12B1) -> BATTERY_-
- J1 pad B6: unconnected-(J1-D+-PadB6) -> USB_D+
- J1 pad B7: unconnected-(J1-D--PadB7) -> USB_D-
- J1 pad B9A4: Net-(J1-VBUS-PadA9B4) -> 5v_Input
- J1 pad S1: unconnected-(J1-SHIELD-PadS1) -> BATTERY_-
- U1 pad 1: unconnected-(U1-LNA_IN-Pad1) -> Net-(U1-LNA_IN)
- U1 pad 11: unconnected-(U1-VDD3P3_RTC-Pad11) -> +3.3V
- U1 pad 14: unconnected-(U1-GPIO8-Pad14) -> SDA
- U1 pad 15: unconnected-(U1-GPIO9-Pad15) -> SCL
- U1 pad 16: unconnected-(U1-GPIO10-Pad16) -> Net-(U1-GPIO10)
- U1 pad 17: unconnected-(U1-VDD3P3_CPU-Pad17) -> +3.3V
- U1 pad 18: unconnected-(U1-(OUTPUT)_VDD_SPI-Pad18) -> VDD_SPI
- U1 pad 19: unconnected-(U1-SPIHD-Pad19) -> SPIHD
- U1 pad 2: Net-(U1-VDD3P3-Pad2) -> +3.3V
- U1 pad 20: unconnected-(U1-SPIWP-Pad20) -> SPIWP
- U1 pad 21: unconnected-(U1-SPICS0-Pad21) -> SPICS0
- U1 pad 22: unconnected-(U1-SPICLK-Pad22) -> SPICLK
- U1 pad 23: unconnected-(U1-SPID-Pad23) -> SPID
- U1 pad 24: unconnected-(U1-SPIQ-Pad24) -> SPIQ
- U1 pad 25: unconnected-(U1-GPIO18/USB_D--Pad25) -> USB_D-
- U1 pad 26: unconnected-(U1-GPIO19/USB_D+-Pad26) -> USB_D+
- U1 pad 29: unconnected-(U1-XTAL_N-Pad29) -> XTAL_N
- U1 pad 3: Net-(U1-VDD3P3-Pad2) -> +3.3V
- U1 pad 30: unconnected-(U1-XTAL_P-Pad30) -> XTAL_P
- U1 pad 31: Net-(U1-VDDA-Pad31) -> +3.3V
- U1 pad 32: Net-(U1-VDDA-Pad31) -> +3.3V
- U1 pad 33: unconnected-(U1-GND-Pad33) -> BATTERY_-
- U1 pad 6: unconnected-(U1-GPIO2-Pad6) -> BATT_SENSOR
- U1 pad 7: unconnected-(U1-CHIP_EN-Pad7) -> +3.3V
- U1 pad 8: unconnected-(U1-GPIO3-Pad8) -> XSHUT
- U2 pad 2: unconnected-(U2-RI-Pad2) -> Net-(U2-PROG)
- U2 pad 3: unconnected-(U2-GND-Pad3) -> BATTERY_-
- U2 pad 4: unconnected-(U2-D+-Pad4) -> 5v_Input
- U2 pad 5: unconnected-(U2-D--Pad5) -> BATTERY_+
- U2 pad 6: unconnected-(U2-VDD-Pad6) -> Net-(U2-STDBY#)
- U2 pad 7: unconnected-(U2-REGIN-Pad7) -> Net-(U2-CHRG#)
- U2 pad 8: unconnected-(U2-VBUS-Pad8) -> 5v_Input
- U2 pad 9: unconnected-(U2-RST#-Pad9) -> BATTERY_-
- U3 pad 1: unconnected-(U3-AVDDVCSEL-Pad1) -> +3.3V
- U3 pad 10: unconnected-(U3-SCL-Pad10) -> SCL
- U3 pad 11: unconnected-(U3-AVDD-Pad11) -> +3.3V
- U3 pad 12: Net-(U3-GND-Pad12) -> BATTERY_-
- U3 pad 2: unconnected-(U3-AVSSVCSEL-Pad2) -> BATTERY_-
- U3 pad 3: Net-(U3-GND-Pad12) -> BATTERY_-
- U3 pad 4: Net-(U3-GND-Pad12) -> BATTERY_-
- U3 pad 5: unconnected-(U3-XSHUT-Pad5) -> XSHUT
- U3 pad 6: Net-(U3-GND-Pad12) -> BATTERY_-
- U3 pad 9: unconnected-(U3-SDA-Pad9) -> SDA
Routing:
- net BATTERY_-: track 0.00 -> 94.8 mm, vias 0 -> 5
- net +3.3V: track 0.00 -> 71.1 mm, vias 0 -> 8
- net 5v_Input: track 0.00 -> 47.6 mm, vias 0 -> 3
- net USB_D-: track 0.00 -> 35.1 mm, vias 0 -> 2
- net XSHUT: track 0.00 -> 32.8 mm, vias 0 -> 2
- net USB_D+: track 0.00 -> 28.0 mm, vias 0 -> 2
- net Net-(U1-LNA_IN): track 0.00 -> 24.1 mm, vias 0 -> 4
- net BATT_SENSOR: track 0.00 -> 23.2 mm, vias 0 -> 2
- net BATTERY_+: track 0.00 -> 20.2 mm, vias 0 -> 3
- net XTAL_N: track 0.00 -> 17.9 mm, vias 0 -> 2
- net Net-(U1-GPIO10): track 0.00 -> 17.7 mm, vias 0 -> 2
- net XTAL_P: track 0.00 -> 17.6 mm, vias 0 -> 2
- net Net-(D3-Pad1): track 0.00 -> 16.7 mm, vias 0 -> 2
- net SDA: track 0.00 -> 16.5 mm, vias 0 -> 2
- net SPIQ: track 0.00 -> 15.3 mm, vias 0 -> 2
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- added copper zone on B.Cu, net BATTERY_-
- added copper zone on F.Cu, net BATTERY_-
Other:
- outline, holes or cut-outs redrawn
- board text added: "+"
- board text added: "-"

Commit message: 20th, January. 2026
Parts:
- removed D3: LTST-C191KRKT, LTST-C191KRKT:0603
- removed R8: 330Ω, PCM_JLCPCB:R_0402
- added S1: EVQ-P3401P, EVQ-P3401P:SW_EVQ-P3401P, F.Cu at (91.0, 76.5)
- U3: value VL53L0CXV0DH1 -> VL53L1CXV0FY1
- moved C4 50.4 mm to (91.3, 72.8)
- moved C7 50.3 mm to (106.1, 63.5)
- moved L1 50.3 mm to (86.6, 68.2)
- moved R1 50.3 mm to (104.6, 63.2)
- moved C1 50.3 mm to (90.1, 68.6)
- moved C3 50.3 mm to (101.7, 66.4)
- moved C5 50.3 mm to (108.3, 63.7)
- moved C6 50.3 mm to (99.3, 61.2)
- moved D1 50.3 mm to (104.8, 67.5)
- moved D2 50.3 mm to (104.8, 66.0)
- moved J2 50.3 mm to (93.3, 70.6)
- moved R10 50.3 mm to (101.7, 64.5)
- moved R2 50.3 mm to (103.3, 63.2)
- moved R4 50.3 mm to (99.3, 60.1)
- moved R5 50.3 mm to (98.7, 58.4)
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Routing:
- net Net-(D3-Pad1): track 16.7 -> 0.00 mm, vias 2 -> 0
- net BATTERY_-: track 94.8 -> 101.7 mm, vias 5 -> 6
- net 5v_Input: track 47.6 -> 49.7 mm
- net XSHUT: track 32.8 -> 31.1 mm
- net USB_D-: track 35.1 -> 33.7 mm
- net Net-(U1-GPIO10): track 17.7 -> 19.0 mm
- net XTAL_N: track 17.9 -> 16.9 mm
- net XTAL_P: track 17.6 -> 16.6 mm
- net Net-(U1-LNA_IN): track 24.1 -> 23.3 mm
- removed copper zone on B.Cu, net BATTERY_-
Other:
- outline, holes or cut-outs redrawn
