File: Waterproof_MEMS_Audio_Logger/Daughter_Board/Daughter_Board/Daughter_Board.kicad_pcb (KiCad board)
At the start: 2 copper layers, 109 x 40 mm, 44 parts, among them J1 S3B-ZR-SM4A-TF, J2 PPTC241LFBN-RC, J3 22-23-2061, U1 STM32G071CBU6, U2 W25Q64JVSSIQ, U3 TPS7A1118PDRVR, X1 X322516MLB4SI

Commit message: 20th, January. 2026
Parts:
- added H1: MountingHole_Pad, MountingHole:MountingHole_4mm_Pad_Via, F.Cu at (102.2, 138.2)
- added H2: MountingHole_Pad, MountingHole:MountingHole_4mm_Pad_Via, F.Cu at (187.2, 138.1)
- added J1: S3B-ZR-SM4A-TF, S3B-ZR-SM4A-TF:JST_S3B-ZR-SM4A-TF, B.Cu at (169.1, 145.9)
- added MK1: AMM-2742-T-WP-R, AMM-2742-T-WP-R:MIC_AMM-2742-T-WP-R, F.Cu at (144.7, 138.1)
Routing:
- net +1V8: track 71.1 -> 105.2 mm, vias 2 -> 3
- net Net-(MK1-DATA): track 0.00 -> 32.6 mm, vias 0 -> 1
- net GND: track 0.00 -> 26.5 mm, vias 0 -> 1
- added copper zone on B.Cu, net GND
- added copper zone on F.Cu, net GND
Other:
- board size 109 x 40 mm -> 109 x 67.2 mm
