File: Waterproof_MEMS_Audio_Logger/Daughter_Board/Daughter_Board/MEMS mic/MEMS mic.kicad_pcb (KiCad board)
At the start: 2 copper layers, 100 x 20 mm, 4 parts, among them J1 S3B-ZR-SM4A-TF

Commit message: 20th, January. 2026
Parts:
- removed MK1: AMM-2742-T-WP-R, AMM-2742-T-WP-R:MIC_AMM-2742-T-WP-R
- added REF**: SolderWirePad_1x01_SMD_5x10mm, Connector_Wire:SolderWirePad_1x01_SMD_5x10mm, F.Cu at (126.0, 93.9)
- added REF**: SolderWirePad_1x01_SMD_5x10mm, Connector_Wire:SolderWirePad_1x01_SMD_5x10mm, F.Cu at (126.0, 97.7)
- added REF**: SolderWirePad_1x01_SMD_5x10mm, Connector_Wire:SolderWirePad_1x01_SMD_5x10mm, F.Cu at (126.0, 90.2)
Routing:
- net GND: track 26.5 -> 72.0 mm
- net Net-(MK1-DATA): track 32.6 -> 69.6 mm
- net +1V8: track 34.1 -> 68.2 mm
Other:
- outline, holes or cut-outs redrawn
